Commit message: save

File: src/kernwald_description/urdf/common_properties.xacro (robot description, xacro)
@@ -14,3 +14,30 @@
         <color rgba="0. 0.6 0 1" />
     </material>
+    <!-- Macroses -->
+    <xacro:macro name="box_inertial" params="mass x y z origin_xyz">
+        <inertial>
+            <origin xyz="${origin_xyz}" rpy="0 0 0" />
+            <mass value="${mass}" />
+            <inertia
+                ixx="${mass / 12.0 * (y * y + z * z)}"
+                ixy="0.0"
+                ixz="0.0"
+                iyy="${mass / 12.0 * (x * x + z * z)}"
+                iyz="0.0"
+                izz="${mass / 12.0 * (x * x + y * y)}" />
+        </inertial>
+    </xacro:macro>
+    <xacro:macro name="cylinder_inertial" params="mass radius length origin_xyz">
+        <inertial>
+            <origin xyz="${origin_xyz}" rpy="0 0 0" />
+            <mass value="${mass}" />
+            <inertia
+                ixx="${mass / 12.0 * (3.0 * radius * radius + length * length)}"
+                ixy="0.0"
+                ixz="0.0"
+                iyy="${mass / 12.0 * (3.0 * radius * radius + length * length)}"
+                iyz="0.0"
+                izz="${mass / 2.0 * radius * radius}" />
+        </inertial>
+    </xacro:macro>
 </robot>

File: src/kernwald_description/urdf/gripper.xacro (robot description, xacro)
@@ -7,4 +7,5 @@
     </joint>
     <link name="gripper_base_link">
+        <xacro:box_inertial mass="0.25" x="0.2" y="0.06" z="0.02" origin_xyz="0 0 0.01" />
         <visual>
             <geometry>
@@ -25,4 +26,5 @@
     </joint>
     <link name="right_finger_link">
+        <xacro:box_inertial mass="0.08" x="0.02" y="0.06" z="0.08" origin_xyz="0 0 0.04" />
         <visual>
             <geometry>
@@ -48,4 +50,5 @@
     </joint>
     <link name="left_finger_link">
+        <xacro:box_inertial mass="0.08" x="0.02" y="0.06" z="0.08" origin_xyz="0 0 0.04" />
         <visual>
             <geometry>

File: src/kernwald_description/urdf/kernwald.ros2_control.xacro (robot description, xacro)
@@ -1,53 +1,59 @@
 <?xml version="1.0"?>
 <robot xmlns:xacro="http://www.ros.org/wiki/xacro">
-    <xacro:property name="initial_positions"
-        value="${xacro.load_yaml(initial_positions_file)['initial_positions']}" />
-    <ros2_control name="KernwaldArm" type="system">
-        <hardware>
-            <!-- By default, set up controllers for simulation. This won't work on real hardware -->
-            <plugin>mock_components/GenericSystem</plugin>
-        </hardware>
-        <joint name="joint_1">
-            <command_interface name="position" />
-            <state_interface name="position">
-                <param name="initial_value">0.0</param>
-            </state_interface>
-        </joint>
-        <joint name="joint_2">
-            <command_interface name="position" />
-            <state_interface name="position">
-                <param name="initial_value">0.0</param>
-            </state_interface>
-        </joint>
-        <joint name="joint_3">
-            <command_interface name="position" />
-            <state_interface name="position">
-                <param name="initial_value">0.0</param>
-            </state_interface>
-        </joint>
-        <joint name="joint_4">
-            <command_interface name="position" />
-            <state_interface name="position">
-                <param name="initial_value">0.0</param>
-            </state_interface>
-        </joint>
-        <joint name="joint_5">
-            <command_interface name="position" />
-            <state_interface name="position">
-                <param name="initial_value">0.0</param>
-            </state_interface>
-        </joint>
-        <joint name="joint_6">
-            <command_interface name="position" />
-            <state_interface name="position">
-                <param name="initial_value">0.0</param>
-            </state_interface>
-        </joint>
-        <joint name="left_finger_joint">
-            <command_interface name="position" />
-            <state_interface name="position">
-                <param name="initial_value">0.0</param>
-            </state_interface>
-        </joint>
-    </ros2_control>
+    <xacro:macro name="kernwald_ros2_control" params="use_gazebo">
+        <ros2_control name="KernwaldArm" type="system">
+            <xacro:if value="${use_gazebo}">
+                <hardware>
+                    <plugin>gz_ros2_control/GazeboSimSystem</plugin>
+                </hardware>
+            </xacro:if>
+            <xacro:unless value="${use_gazebo}">
+                <hardware>
+                    <plugin>mock_components/GenericSystem</plugin>
+                </hardware>
+            </xacro:unless>
+            <joint name="joint_1">
+                <command_interface name="position" />
+                <state_interface name="position">
+                    <param name="initial_value">0.0</param>
+                </state_interface>
+            </joint>
+            <joint name="joint_2">
+                <command_interface name="position" />
+                <state_interface name="position">
+                    <param name="initial_value">0.0</param>
+                </state_interface>
+            </joint>
+            <joint name="joint_3">
+                <command_interface name="position" />
+                <state_interface name="position">
+                    <param name="initial_value">0.0</param>
+                </state_interface>
+            </joint>
+            <joint name="joint_4">
+                <command_interface name="position" />
+                <state_interface name="position">
+                    <param name="initial_value">0.0</param>
+                </state_interface>
+            </joint>
+            <joint name="joint_5">
+                <command_interface name="position" />
+                <state_interface name="position">
+                    <param name="initial_value">0.0</param>
+                </state_interface>
+            </joint>
+            <joint name="joint_6">
+                <command_interface name="position" />
+                <state_interface name="position">
+                    <param name="initial_value">0.0</param>
+                </state_interface>
+            </joint>
+            <joint name="left_finger_joint">
+                <command_interface name="position" />
+                <state_interface name="position">
+                    <param name="initial_value">0.0</param>
+                </state_interface>
+            </joint>
+        </ros2_control>
+    </xacro:macro>
 </robot>

File: src/kernwald_description/urdf/kernwald.xacro (robot description, xacro)
@@ -3,6 +3,18 @@
     <!-- Includes -->
     <xacro:include filename="common_properties.xacro" />
+    <xacro:include filename="kernwald.ros2_control.xacro" />
+    <xacro:arg name="use_gazebo" default="false" />
+    <xacro:arg name="controllers_file" default="" />
     <xacro:include filename="gripper.xacro" />
+    <xacro:kernwald_ros2_control use_gazebo="$(arg use_gazebo)" />
+    <!-- Base -->
+    <link name="base_footprint" />
+    <joint name="base_footprint_joint" type="fixed">
+        <parent link="base_footprint" />
+        <child link="base_link" />
+        <origin xyz="0 0 0" rpy="0 0 0" />
+    </joint>
     <link name="base_link">
+        <xacro:box_inertial mass="5.0" x="0.4" y="0.4" z="0.1" origin_xyz="0 0 0.05" />
         <visual>
             <geometry>
@@ -28,4 +40,5 @@
     </joint>
     <link name="shoulder_link">
+        <xacro:cylinder_inertial mass="2.0" radius="0.1" length="0.5" origin_xyz="0 0 0.25" />
         <visual>
             <geometry>
@@ -51,4 +64,5 @@
     </joint>
     <link name="arm_link">
+        <xacro:cylinder_inertial mass="1.5" radius="0.05" length="0.6" origin_xyz="0 0 0.3" />
         <visual>
             <geometry>
@@ -74,4 +88,5 @@
     </joint>
     <link name="elbow_link">
+        <xacro:cylinder_inertial mass="0.5" radius="0.05" length="0.1" origin_xyz="0 0 0.05" />
         <visual>
             <geometry>
@@ -97,4 +112,5 @@
     </joint>
     <link name="forearm_link">
+        <xacro:cylinder_inertial mass="1.0" radius="0.05" length="0.5" origin_xyz="0 0 0.25" />
         <visual>
             <geometry>
@@ -120,4 +136,5 @@
     </joint>
     <link name="wrist_link">
+        <xacro:box_inertial mass="0.4" x="0.1" y="0.1" z="0.05" origin_xyz="0 0 0.025" />
         <visual>
             <geometry>
@@ -143,4 +160,5 @@
     </joint>
     <link name="hand_link">
+        <xacro:box_inertial mass="0.2" x="0.1" y="0.1" z="0.02" origin_xyz="0 0 0.01" />
         <visual>
             <geometry>
@@ -163,6 +181,15 @@
         <origin xyz="0 0 0.02" rpy="0 0 0" />
     </joint>
-    <link name="tool_link" />
-    <!-- Import control_xacro -->
-    <xacro:include filename="kernwald.ros2_control.xacro" />
+    <link name="tool_link">
+        <xacro:box_inertial mass="0.05" x="0.02" y="0.02" z="0.02" origin_xyz="0 0 0" />
+    </link>
+    <!-- Gazebo -->
+    <xacro:if value="$(arg use_gazebo)">
+        <gazebo>
+            <plugin filename="libgz_ros2_control-system.so"
+                name="gz_ros2_control::GazeboSimROS2ControlPlugin">
+                <parameters>$(arg controllers_file)</parameters>
+            </plugin>
+        </gazebo>
+    </xacro:if>
 </robot>

File: src/kernwalt_moveit_config/config/kernwald.ros2_control.xacro (robot description, xacro)
@@ -1,51 +1,60 @@
 <?xml version="1.0"?>
 <robot xmlns:xacro="http://www.ros.org/wiki/xacro">
-    <xacro:macro name="kernwald_ros2_control" params="name initial_positions_file">
-        <xacro:property name="initial_positions" value="${xacro.load_yaml(initial_positions_file)['initial_positions']}"/>
+    <xacro:macro name="kernwald_ros2_control" params="name initial_positions_file use_gazebo">
+        <xacro:property name="initial_positions"
+            value="${xacro.load_yaml(initial_positions_file)['initial_positions']}" />
         <ros2_control name="${name}" type="system">
-            <hardware>
-                <!-- By default, set up controllers for simulation. This won't work on real hardware -->
-                <plugin>mock_components/GenericSystem</plugin>
-            </hardware>
+            <xacro:if value="${use_gazebo}">
+                <hardware>
+                    <plugin>gz_ros2_control/GazeboSimSystem</plugin>
+                </hardware>
+            </xacro:if>
+            <xacro:unless value="${use_gazebo}">
+                <hardware>
+                    <!-- By default, set up controllers for simulation. This won't work on real
+                    hardware -->
+                    <plugin>mock_components/GenericSystem</plugin>
+                </hardware>
+            </xacro:unless>
             <joint name="joint_1">
-                <command_interface name="position"/>
+                <command_interface name="position" />
                 <state_interface name="position">
-                  <param name="initial_value">${initial_positions['joint_1']}</param>
+                    <param name="initial_value">${initial_positions['joint_1']}</param>
                 </state_interface>
             </joint>
             <joint name="joint_2">
-                <command_interface name="position"/>
+                <command_interface name="position" />
                 <state_interface name="position">
-                  <param name="initial_value">${initial_positions['joint_2']}</param>
+                    <param name="initial_value">${initial_positions['joint_2']}</param>
                 </state_interface>
             </joint>
             <joint name="joint_3">
-                <command_interface name="position"/>
+                <command_interface name="position" />
                 <state_interface name="position">
-                  <param name="initial_value">${initial_positions['joint_3']}</param>
+                    <param name="initial_value">${initial_positions['joint_3']}</param>
                 </state_interface>
             </joint>
             <joint name="joint_4">
-                <command_interface name="position"/>
+                <command_interface name="position" />
                 <state_interface name="position">
-                  <param name="initial_value">${initial_positions['joint_4']}</param>
+                    <param name="initial_value">${initial_positions['joint_4']}</param>
                 </state_interface>
             </joint>
             <joint name="joint_5">
-                <command_interface name="position"/>
+                <command_interface name="position" />
                 <state_interface name="position">
-                  <param name="initial_value">${initial_positions['joint_5']}</param>
+                    <param name="initial_value">${initial_positions['joint_5']}</param>
                 </state_interface>
             </joint>
             <joint name="joint_6">
-                <command_interface name="position"/>
+                <command_interface name="position" />
                 <state_interface name="position">
-                  <param name="initial_value">${initial_positions['joint_6']}</param>
+                    <param name="initial_value">${initial_positions['joint_6']}</param>
                 </state_interface>
             </joint>
             <joint name="left_finger_joint">
-                <command_interface name="position"/>
+                <command_interface name="position" />
                 <state_interface name="position">
-                  <param name="initial_value">${initial_positions['left_finger_joint']}</param>
+                    <param name="initial_value">${initial_positions['left_finger_joint']}</param>
                 </state_interface>
             </joint>

File: src/kernwalt_moveit_config/config/kernwald.urdf.xacro (robot description, xacro)
@@ -4,6 +4,3 @@
     <!-- Import kernwald urdf file -->
     <xacro:include filename="$(find kernwald_description)/urdf/kernwald.xacro" />
-    <!-- Import control_xacro -->
-    <xacro:include filename="kernwald.ros2_control.xacro" />
-    <xacro:kernwald_ros2_control name="FakeSystem" initial_positions_file="$(arg initial_positions_file)"/>
 </robot>
