Commit message: checkpoint

File: src/kernwald_description/urdf/kernwald.ros2_control.xacro (robot description, xacro)
@@ -55,4 +55,11 @@
                 </state_interface>
             </joint>
+            <joint name="right_finger_joint">
+                <param name="mimic">left_finger_joint</param>
+                <param name="multiplier">-1.0</param>
+                <state_interface name="position">
+                    <param name="initial_value">0.0</param>
+                </state_interface>
+            </joint>
         </ros2_control>
     </xacro:macro>

File: src/kernwald_description/urdf/kernwald.xacro (robot description, xacro)
@@ -183,10 +183,12 @@
         <xacro:box_inertial mass="0.05" x="0.02" y="0.02" z="0.02" origin_xyz="0 0 0" />
     </link>
-    <!-- Gazebo -->
-    <gazebo>
-        <plugin filename="libgz_ros2_control-system.so"
-            name="gz_ros2_control::GazeboSimROS2ControlPlugin">
-            <parameters>$(find kernwald_bringup)/config/ros2_controllers.yaml</parameters>
-        </plugin>
-    </gazebo>
+    <xacro:if value="$(arg use_gazebo)">
+        <!-- Gazebo -->
+        <gazebo>
+            <plugin filename="libgz_ros2_control-system.so"
+                name="gz_ros2_control::GazeboSimROS2ControlPlugin">
+                <parameters>$(find kernwald_bringup)/config/ros2_controllers.yaml</parameters>
+            </plugin>
+        </gazebo>
+    </xacro:if>
 </robot>

File: src/kernwalt_moveit_config/config/kernwald.ros2_control.xacro (robot description, xacro)
@@ -59,4 +59,11 @@
                 </state_interface>
             </joint>
+            <joint name="right_finger_joint">
+                <param name="mimic">left_finger_joint</param>
+                <param name="multiplier">-1.0</param>
+                <state_interface name="position">
+                    <param name="initial_value">${initial_positions['left_finger_joint'] * -1.0}</param>
+                </state_interface>
+            </joint>
         </ros2_control>
     </xacro:macro>
