Commit message: Porting gazebo

File: src/kernwald_description/urdf/gripper.xacro (robot description, xacro)
@@ -21,7 +21,6 @@
         <child link="right_finger_link" />
         <origin xyz="0.07 0 0.02" rpy="0 0 0" />
-        <axis xyz="1 0 0" />
-        <limit effort="1000.0" velocity="1.0" lower="-0.06" upper="0.0" />
-        <mimic joint="left_finger_joint" multiplier="-1.0" />
+        <axis xyz="-1 0 0" />
+        <limit effort="1000.0" velocity="1.0" lower="-0.001" upper="0.06" />
     </joint>
     <link name="right_finger_link">
@@ -47,5 +46,5 @@
         <origin xyz="-0.07 0 0.02" rpy="0 0 0" />
         <axis xyz="1 0 0" />
-        <limit effort="1000.0" velocity="1.0" lower="0.0" upper="0.06" />
+        <limit effort="1000.0" velocity="1.0" lower="-0.001" upper="0.06" />
     </joint>
     <link name="left_finger_link">

File: src/kernwald_description/urdf/kernwald.ros2_control.xacro (robot description, xacro)
@@ -56,6 +56,5 @@
             </joint>
             <joint name="right_finger_joint">
-                <param name="mimic">left_finger_joint</param>
-                <param name="multiplier">-1.0</param>
+                <command_interface name="position" />
                 <state_interface name="position">
                     <param name="initial_value">0.0</param>

File: src/kernwalt_moveit_config/config/kernwald.ros2_control.xacro (robot description, xacro)
@@ -60,8 +60,7 @@
             </joint>
             <joint name="right_finger_joint">
-                <param name="mimic">left_finger_joint</param>
-                <param name="multiplier">-1.0</param>
+                <command_interface name="position" />
                 <state_interface name="position">
-                    <param name="initial_value">${initial_positions['left_finger_joint'] * -1.0}</param>
+                    <param name="initial_value">${initial_positions['right_finger_joint']}</param>
                 </state_interface>
             </joint>
