Commit message: add depth camera & planning scene

File: src/kernwald_description/urdf/kernwald.xacro (robot description, xacro)
@@ -183,4 +183,49 @@
         <xacro:box_inertial mass="0.05" x="0.02" y="0.02" z="0.02" origin_xyz="0 0 0" />
     </link>
+    <!-- Overhead depth camera -->
+    <joint name="depth_camera_joint" type="fixed">
+        <parent link="base_footprint" />
+        <child link="depth_camera_link" />
+        <origin xyz="0.15 0 2.5" rpy="0 1.5708 0" />
+    </joint>
+    <link name="depth_camera_link">
+        <xacro:box_inertial mass="0.1" x="0.06" y="0.06" z="0.04" origin_xyz="0 0 0" />
+        <visual>
+            <geometry>
+                <box size="0.06 0.06 0.04" />
+            </geometry>
+            <origin xyz="0 0 0" rpy="0 0 0" />
+            <material name="grey" />
+        </visual>
+        <collision>
+            <geometry>
+                <box size="0.06 0.06 0.04" />
+            </geometry>
+            <origin xyz="0 0 0" rpy="0 0 0" />
+        </collision>
+    </link>
+    <xacro:if value="$(arg use_gazebo)">
+        <gazebo reference="depth_camera_link">
+            <sensor name="depth_camera" type="depth_camera">
+                <always_on>true</always_on>
+                <update_rate>10</update_rate>
+                <topic>depth_camera</topic>
+                <frame_id>depth_camera_link</frame_id>
+                <camera>
+                    <horizontal_fov>1.9</horizontal_fov>
+                    <optical_frame_id>depth_camera_link</optical_frame_id>
+                    <image>
+                        <width>424</width>
+                        <height>240</height>
+                        <format>R8G8B8</format>
+                    </image>
+                    <clip>
+                        <near>0.2</near>
+                        <far>6.0</far>
+                    </clip>
+                </camera>
+            </sensor>
+        </gazebo>
+    </xacro:if>
     <xacro:if value="$(arg use_gazebo)">
         <!-- Gazebo -->
